Commit message: working

File: body.urdf (robot description, URDF)
Before this commit: robot robot, 3 links, 2 joints
Links:
- added link BackLowerLeg, mass 1; collision box size=0.2 0.2 1; visual box size=0.2 0.2 1
- added link FrontLowerLeg, mass 1; collision box size=0.2 0.2 1; visual box size=0.2 0.2 1
- added link LeftLeg, mass 1; collision box size=1 0.2 0.2; visual box size=1 0.2 0.2
- added link LeftLowerLeg, mass 1; collision box size=0.2 0.2 1; visual box size=0.2 0.2 1
- added link RightLeg, mass 1; collision box size=1 0.2 0.2; visual box size=1 0.2 0.2
- added link RightLowerLeg, mass 1; collision box size=0.2 0.2 1; visual box size=0.2 0.2 1
- link BackLeg: geometry collision box size=0.2 1 0.2; visual box size=0.2 1 0.2
- link FrontLeg: geometry collision box size=0.2 1 0.2; visual box size=0.2 1 0.2
Joints:
- added joint BackLeg_BackLowerLeg: type revolute, parent BackLeg, child BackLowerLeg, origin xyz=0 1 0 rpy=0 0 0, axis 1 0 0, limit lower=-3.14159 upper=3.14159 effort=0.0 velocity=0.0
- added joint FrontLeg_FrontLowerLeg: type revolute, parent FrontLeg, child FrontLowerLeg, origin xyz=0 1 0 rpy=0 0 0, axis 1 0 0, limit lower=-3.14159 upper=3.14159 effort=0.0 velocity=0.0
- added joint LeftLeg_LeftLowerLeg: type revolute, parent LeftLeg, child LeftLowerLeg, origin xyz=0 1 0 rpy=0 0 0, axis 1 0 0, limit lower=-3.14159 upper=3.14159 effort=0.0 velocity=0.0
- added joint RightLeg_RightLowerLeg: type revolute, parent RightLeg, child RightLowerLeg, origin xyz=0 1 0 rpy=0 0 0, axis 1 0 0, limit lower=-3.14159 upper=3.14159 effort=0.0 velocity=0.0
- added joint Torso_LeftLeg: type revolute, parent Torso, child LeftLeg, origin xyz=-0.5 0 1 rpy=0 0 0, axis 0 1 0, limit lower=-3.14159 upper=3.14159 effort=0.0 velocity=0.0
- added joint Torso_RightLeg: type revolute, parent Torso, child RightLeg, origin xyz=0.5 0 1 rpy=0 0 0, axis 0 1 0, limit lower=-3.14159 upper=3.14159 effort=0.0 velocity=0.0
- joint Torso_BackLeg: axis 0 1 0 -> 1 0 0; origin xyz=1 0 1 rpy=0 0 0 -> xyz=0 -0.5 1 rpy=0 0 0
- joint Torso_FrontLeg: axis 0 1 0 -> 1 0 0; origin xyz=2 0 1 rpy=0 0 0 -> xyz=0 0.5 1 rpy=0 0 0

Commit message: almost there

File: body.urdf (robot description, URDF)
Before this commit: robot robot, 9 links, 8 joints
Joints:
- joint BackLeg_BackLowerLeg: origin xyz=0 1 0 rpy=0 0 0 -> xyz=0 -1 0 rpy=0 0 0
- joint LeftLeg_LeftLowerLeg: axis 1 0 0 -> 0 1 0; origin xyz=0 1 0 rpy=0 0 0 -> xyz=-1 0 0 rpy=0 0 0
- joint RightLeg_RightLowerLeg: axis 1 0 0 -> 0  1 0; origin xyz=0 1 0 rpy=0 0 0 -> xyz=1 0 0 rpy=0 0 0

Commit message: robot with a ball

File: body.urdf (robot description, URDF)
Before this commit: robot robot, 9 links, 8 joints
Links:
- removed link BackLeg
- removed link BackLowerLeg
- removed link FrontLeg
- removed link FrontLowerLeg
- removed link LeftLowerLeg
- removed link RightLowerLeg
- added link Head, mass 1; collision box size=0.4 0.4 0.5; visual box size=0.4 0.4 0.5
- link LeftLeg: geometry collision box size=0.4 0.4 1.25; visual box size=0.4 0.4 1.25
- link RightLeg: geometry collision box size=0.4 0.4 1.25; visual box size=0.4 0.4 1.25
- link Torso: geometry collision box size=0.75 0.4 1; visual box size=0.75 0.4 1
Joints:
- removed joint BackLeg_BackLowerLeg
- removed joint FrontLeg_FrontLowerLeg
- removed joint LeftLeg_LeftLowerLeg
- removed joint RightLeg_RightLowerLeg
- removed joint Torso_BackLeg
- removed joint Torso_FrontLeg
- added joint Torso_Head: type revolute, parent Torso, child Head, origin xyz=0 0 2.1 rpy=0 0 0, axis 1 0 0, limit lower=-3.14159 upper=3.14159 effort=0.0 velocity=0.0
- joint Torso_LeftLeg: axis 0 1 0 -> 1 0 0; origin xyz=-0.5 0 1 rpy=0 0 0 -> xyz=-0.375 0 1.25 rpy=0 0 0
- joint Torso_RightLeg: axis 0 1 0 -> 1 0 0; origin xyz=0.5 0 1 rpy=0 0 0 -> xyz=0.375 0 1.25 rpy=0 0 0

Commit message: robot kicks!

File: body.urdf (robot description, URDF)
Before this commit: robot robot, 4 links, 3 joints
Links:
- added link LeftArm, mass 1; collision box size=0.2 0.4 0.6; visual box size=0.2 0.4 0.6
- added link LeftShoulder, mass 1; collision box size=0.3 0.4 0.2; visual box size=0.3 0.4 0.2
- added link RightArm, mass 1; collision box size=0.2 0.4 0.6; visual box size=0.2 0.4 0.6
- added link RightShoulder, mass 1; collision box size=0.3 0.4 0.2; visual box size=0.3 0.4 0.2
- link Head: geometry collision box size=0.4 0.4 0.4; visual box size=0.4 0.4 0.4
Joints:
- added joint LeftShoulder_LeftArm: type revolute, parent LeftShoulder, child LeftArm, origin xyz=-0.3 0 0 rpy=0 0 0, axis 1 0 0, limit lower=-3.14159 upper=3.14159 effort=0.0 velocity=0.0
- added joint RightShoulder_RightArm: type revolute, parent RightShoulder, child RightArm, origin xyz=0.3 0 0 rpy=0 0 0, axis 1 0 0, limit lower=-3.14159 upper=3.14159 effort=0.0 velocity=0.0
- added joint Torso_LeftShoulder: type revolute, parent Torso, child LeftShoulder, origin xyz=-0.2 0 2.05 rpy=0 0 0, axis 1 0 0, limit lower=-3.14159 upper=3.14159 effort=0.0 velocity=0.0
- added joint Torso_RightShoulder: type revolute, parent Torso, child RightShoulder, origin xyz=0.2 0 2.05 rpy=0 0 0, axis 1 0 0, limit lower=-3.14159 upper=3.14159 effort=0.0 velocity=0.0

Commit message: created snake, debugging

File: body.urdf (robot description, URDF)
Before this commit: robot robot, 8 links, 7 joints
Links:
- removed link Head
- removed link LeftArm
- removed link LeftLeg
- removed link LeftShoulder
- removed link RightArm
- removed link RightLeg
- removed link RightShoulder
- removed link Torso
- added link Link0, mass 1; collision box size=0.355193781593668 0.49223529130993615 0.4240798974658009; visual box size=0.355193781593668 0.49223529130993615 0.4240798974658009
- added link Link1, mass 1; collision box size=0.7379497386931168 0.8858264790244466 0.5658734743122783; visual box size=0.7379497386931168 0.8858264790244466 0.5658734743122783
- added link Link2, mass 1; collision box size=0.8517138932455901 0.8142456743702844 0.49970717036167656; visual box size=0.8517138932455901 0.8142456743702844 0.49970717036167656
- added link Link3, mass 1; collision box size=0.4167048098319248 1.0654501709781734 0.9482121932670808; visual box size=0.4167048098319248 1.0654501709781734 0.9482121932670808
- added link Link4, mass 1; collision box size=0.9155020357483112 0.27040672606326943 0.3644409270393417; visual box size=0.9155020357483112 0.27040672606326943 0.3644409270393417
- added link Link5, mass 1; collision box size=0.40528452372798873 0.8482796732872951 0.5591746329488699; visual box size=0.40528452372798873 0.8482796732872951 0.5591746329488699
Joints:
- removed joint LeftShoulder_LeftArm
- removed joint RightShoulder_RightArm
- removed joint Torso_Head
- removed joint Torso_LeftLeg
- removed joint Torso_LeftShoulder
- removed joint Torso_RightLeg
- removed joint Torso_RightShoulder
- added joint Link0_Link1: type revolute, parent Link0, child Link1, origin xyz=-0.8224031092031661 0 0 rpy=0 0 0, axis 1 0 0, limit lower=-3.14159 upper=3.14159 effort=0.0 velocity=0.0
- added joint Link1_Link2: type revolute, parent Link1, child Link2, origin xyz=0.7379497386931168 0 0 rpy=0 0 0, axis 1 0 0, limit lower=-3.14159 upper=3.14159 effort=0.0 velocity=0.0
- added joint Link2_Link3: type revolute, parent Link2, child Link3, origin xyz=0.8517138932455901 0 0 rpy=0 0 0, axis 1 0 0, limit lower=-3.14159 upper=3.14159 effort=0.0 velocity=0.0
- added joint Link3_Link4: type revolute, parent Link3, child Link4, origin xyz=0.4167048098319248 0 0 rpy=0 0 0, axis 1 0 0, limit lower=-3.14159 upper=3.14159 effort=0.0 velocity=0.0
- added joint Link4_Link5: type revolute, parent Link4, child Link5, origin xyz=0.9155020357483112 0 0 rpy=0 0 0, axis 1 0 0, limit lower=-3.14159 upper=3.14159 effort=0.0 velocity=0.0

Commit message: finishing a6

File: body.urdf (robot description, URDF)
Before this commit: robot robot, 6 links, 5 joints
Links:
- link Link0: geometry collision box size=0.6777299092870434 0.9228734932345072 0.7656022005149777; visual box size=0.6777299092870434 0.9228734932345072 0.7656022005149777
- link Link1: geometry collision box size=0.9761796737159663 0.9965515214285149 0.3910860552070673; visual box size=0.9761796737159663 0.9965515214285149 0.3910860552070673
- link Link2: geometry collision box size=0.728644724329153 0.2863810834114231 0.23765374158050126; visual box size=0.728644724329153 0.2863810834114231 0.23765374158050126
- link Link3: geometry collision box size=0.16730140566179677 0.35385540637121604 1.0875968828128042; visual box size=0.16730140566179677 0.35385540637121604 1.0875968828128042
- link Link4: geometry collision box size=0.7946478101790576 0.28887694166177436 0.6010002148239135; visual box size=0.7946478101790576 0.28887694166177436 0.6010002148239135
- link Link5: geometry collision box size=0.3023795156142913 0.5095489948459563 0.8365340918536097; visual box size=0.3023795156142913 0.5095489948459563 0.8365340918536097
Joints:
- joint Link0_Link1: origin xyz=-0.8224031092031661 0 0 rpy=0 0 0 -> xyz=-0.6611350453564784 0 0 rpy=0 0 0
- joint Link1_Link2: origin xyz=0.7379497386931168 0 0 rpy=0 0 0 -> xyz=0.9761796737159663 0 0 rpy=0 0 0
- joint Link2_Link3: origin xyz=0.8517138932455901 0 0 rpy=0 0 0 -> xyz=0.728644724329153 0 0 rpy=0 0 0
- joint Link3_Link4: origin xyz=0.4167048098319248 0 0 rpy=0 0 0 -> xyz=0.16730140566179677 0 0 rpy=0 0 0
- joint Link4_Link5: origin xyz=0.9155020357483112 0 0 rpy=0 0 0 -> xyz=0.7946478101790576 0 0 rpy=0 0 0

Commit message: finished assignment 6

File: body.urdf (robot description, URDF)
Before this commit: robot robot, 6 links, 5 joints
Links:
- added link Link6, mass 1; collision box size=0.5511496228527049 0.3034483268355207 0.8181171227530697; visual box size=0.5511496228527049 0.3034483268355207 0.8181171227530697
- added link Link7, mass 1; collision box size=0.11279032168316663 0.13572448728545086 0.5554996193508117; visual box size=0.11279032168316663 0.13572448728545086 0.5554996193508117
- link Link0: geometry collision box size=0.4487425796463489 0.6800941910495247 0.2626974117550285; visual box size=0.4487425796463489 0.6800941910495247 0.2626974117550285
- link Link1: geometry collision box size=0.20924822863935114 0.27719669139557557 0.43563197955149724; visual box size=0.20924822863935114 0.27719669139557557 0.43563197955149724
- link Link2: geometry collision box size=0.13828454518078617 0.22419111936461836 1.0231716362733803; visual box size=0.13828454518078617 0.22419111936461836 1.0231716362733803
- link Link3: geometry collision box size=0.5403503091691984 0.5456287544027516 0.9653924138478179; visual box size=0.5403503091691984 0.5456287544027516 0.9653924138478179
- link Link4: geometry collision box size=0.5686359508373547 0.751950726807557 0.5999467857755618; visual box size=0.5686359508373547 0.751950726807557 0.5999467857755618
- link Link5: geometry collision box size=1.064204686777142 0.7506532756812739 0.36237631206803866; visual box size=1.064204686777142 0.7506532756812739 0.36237631206803866
Joints:
- added joint Link5_Link6: type revolute, parent Link5, child Link6, origin xyz=1.064204686777142 0 0 rpy=0 0 0, axis 1 0 0, limit lower=-3.14159 upper=3.14159 effort=0.0 velocity=0.0
- added joint Link6_Link7: type revolute, parent Link6, child Link7, origin xyz=0.5511496228527049 0 0 rpy=0 0 0, axis 1 0 0, limit lower=-3.14159 upper=3.14159 effort=0.0 velocity=0.0
- joint Link0_Link1: origin xyz=-0.6611350453564784 0 0 rpy=0 0 0 -> xyz=-0.7756287101768256 0 0 rpy=0 0 0
- joint Link1_Link2: origin xyz=0.9761796737159663 0 0 rpy=0 0 0 -> xyz=0.20924822863935114 0 0 rpy=0 0 0
- joint Link2_Link3: origin xyz=0.728644724329153 0 0 rpy=0 0 0 -> xyz=0.13828454518078617 0 0 rpy=0 0 0
- joint Link3_Link4: origin xyz=0.16730140566179677 0 0 rpy=0 0 0 -> xyz=0.5403503091691984 0 0 rpy=0 0 0
- joint Link4_Link5: origin xyz=0.7946478101790576 0 0 rpy=0 0 0 -> xyz=0.5686359508373547 0 0 rpy=0 0 0

Commit message: working on it

File: body.urdf (robot description, URDF)
Before this commit: robot robot, 8 links, 7 joints
Links:
- removed link Link3
- removed link Link4
- removed link Link5
- removed link Link6
- removed link Link7
- link Link0: geometry collision box size=0.9898425728939135 0.4917455728199388 0.8391780992642737; visual box size=0.9898425728939135 0.4917455728199388 0.8391780992642737
- link Link1: geometry collision box size=0.6711185865957466 0.1000558810581548 0.44448266945716775; visual box size=0.6711185865957466 0.1000558810581548 0.44448266945716775
- link Link2: geometry collision box size=0.38062569665828294 0.8090409682558202 0.9431474162364468; visual box size=0.38062569665828294 0.8090409682558202 0.9431474162364468
Joints:
- removed joint Link2_Link3
- removed joint Link3_Link4
- removed joint Link4_Link5
- removed joint Link5_Link6
- removed joint Link6_Link7
- joint Link0_Link1: origin xyz=-0.7756287101768256 0 0 rpy=0 0 0 -> xyz=-1 0.2458727864099694 0.5 rpy=0 0 0
- joint Link1_Link2: origin xyz=0.20924822863935114 0 0 rpy=0 0 0 -> xyz=0 -0.1000558810581548 0 rpy=0 0 0

Commit message: finishing a7

File: body.urdf (robot description, URDF)
Before this commit: robot robot, 3 links, 2 joints
Links:
- added link Link10, mass 1; collision box size=0.7013603132919191 0.6256005661811557 0.6726477803990479; visual box size=0.7013603132919191 0.6256005661811557 0.6726477803990479
- added link Link11, mass 1; collision box size=0.3312007858309678 0.34872597361926694 0.701032694715215; visual box size=0.3312007858309678 0.34872597361926694 0.701032694715215
- added link Link12, mass 1; collision box size=0.10387347648667669 0.5791803905441331 0.20547558738330066; visual box size=0.10387347648667669 0.5791803905441331 0.20547558738330066
- added link Link3, mass 1; collision box size=0.5340228605494286 0.4997182456321605 0.8740269131828778; visual box size=0.5340228605494286 0.4997182456321605 0.8740269131828778
- added link Link4, mass 1; collision box size=1.0581551188462235 0.49542602885079623 0.614500734143948; visual box size=1.0581551188462235 0.49542602885079623 0.614500734143948
- added link Link5, mass 1; collision box size=0.9725421364960399 0.8848313811778493 0.7941157236639428; visual box size=0.9725421364960399 0.8848313811778493 0.7941157236639428
- added link Link6, mass 1; collision box size=0.9949596565867788 0.7440819402699874 0.2611275784815954; visual box size=0.9949596565867788 0.7440819402699874 0.2611275784815954
- added link Link7, mass 1; collision box size=0.17716414715884135 0.8179846961451815 0.7839931310546844; visual box size=0.17716414715884135 0.8179846961451815 0.7839931310546844
- added link Link8, mass 1; collision box size=0.5631107828335741 0.6519226700009095 0.8537247623249259; visual box size=0.5631107828335741 0.6519226700009095 0.8537247623249259
- added link Link9, mass 1; collision box size=0.9503330964372043 0.794041545211034 0.41931308380882715; visual box size=0.9503330964372043 0.794041545211034 0.41931308380882715
- link Link0: geometry collision box size=0.11634581292879256 0.7150914290957515 0.8807051858517716; visual box size=0.11634581292879256 0.7150914290957515 0.8807051858517716
- link Link1: geometry collision box size=0.892626205858006 0.6976178794959438 0.40414343821851706; visual box size=0.892626205858006 0.6976178794959438 0.40414343821851706
- link Link2: geometry collision box size=0.18703109386814523 0.8369508294019093 0.30011200290851814; visual box size=0.18703109386814523 0.8369508294019093 0.30011200290851814
Joints:
- added joint Link10_Link11: type revolute, parent Link10, child Link11, origin xyz=0.35068015664595953 0 0.33632389019952397 rpy=0 0 0, axis 1 0 0, limit lower=-3.14159 upper=3.14159 effort=0.0 velocity=0.0
- added joint Link11_Link12: type revolute, parent Link11, child Link12, origin xyz=0 -0.17436298680963347 0.3505163473576075 rpy=0 0 0, axis 1 0 0, limit lower=-3.14159 upper=3.14159 effort=0.0 velocity=0.0
- added joint Link2_Link3: type revolute, parent Link2, child Link3, origin xyz=0 0.8369508294019093 0 rpy=0 0 0, axis 1 0 0, limit lower=-3.14159 upper=3.14159 effort=0.0 velocity=0.0
- added joint Link3_Link4: type revolute, parent Link3, child Link4, origin xyz=0.2670114302747143 0.24985912281608025 0 rpy=0 0 0, axis 1 0 0, limit lower=-3.14159 upper=3.14159 effort=0.0 velocity=0.0
- added joint Link4_Link5: type revolute, parent Link4, child Link5, origin xyz=0.5290775594231117 0.24771301442539811 0 rpy=0 0 0, axis 1 0 0, limit lower=-3.14159 upper=3.14159 effort=0.0 velocity=0.0
- added joint Link5_Link6: type revolute, parent Link5, child Link6, origin xyz=0 0.8848313811778493 0 rpy=0 0 0, axis 1 0 0, limit lower=-3.14159 upper=3.14159 effort=0.0 velocity=0.0
- added joint Link6_Link7: type revolute, parent Link6, child Link7, origin xyz=0.4974798282933894 0.3720409701349937 0 rpy=0 0 0, axis 1 0 0, limit lower=-3.14159 upper=3.14159 effort=0.0 velocity=0.0
- added joint Link7_Link8: type revolute, parent Link7, child Link8, origin xyz=0.08858207357942068 0.4089923480725908 0 rpy=0 0 0, axis 1 0 0, limit lower=-3.14159 upper=3.14159 effort=0.0 velocity=0.0
- added joint Link8_Link9: type revolute, parent Link8, child Link9, origin xyz=0 0.6519226700009095 0 rpy=0 0 0, axis 1 0 0, limit lower=-3.14159 upper=3.14159 effort=0.0 velocity=0.0
- added joint Link9_Link10: type revolute, parent Link9, child Link10, origin xyz=0.47516654821860216 0.397020772605517 0 rpy=0 0 0, axis 1 0 0, limit lower=-3.14159 upper=3.14159 effort=0.0 velocity=0.0
- joint Link0_Link1: origin xyz=-1 0.2458727864099694 0.5 rpy=0 0 0 -> xyz=-1 -0.35754571454787576 0.5 rpy=0 0 0
- joint Link1_Link2: origin xyz=0 -0.1000558810581548 0 rpy=0 0 0 -> xyz=0 0.6976178794959438 0 rpy=0 0 0

Commit message: debugging

File: body.urdf (robot description, URDF)
Before this commit: robot robot, 13 links, 12 joints
Links:
- removed link Link10
- removed link Link11
- removed link Link12
- removed link Link7
- removed link Link8
- removed link Link9
- link Link0: geometry collision box size=0.24633679041667758 0.9463366869798392 0.7704001125734071; visual box size=0.24633679041667758 0.9463366869798392 0.7704001125734071
- link Link1: geometry collision box size=0.7419446069859255 0.5463345754935891 0.5504892038643788; visual box size=0.7419446069859255 0.5463345754935891 0.5504892038643788
- link Link2: geometry collision box size=0.37540426636480195 0.7855029938258142 1.031789114112372; visual box size=0.37540426636480195 0.7855029938258142 1.031789114112372
- link Link3: geometry collision box size=0.6219746641179585 0.21833596710714767 1.0751778008331214; visual box size=0.6219746641179585 0.21833596710714767 1.0751778008331214
- link Link4: geometry collision box size=0.47245005204754464 0.3340878974221754 0.11994987425580875; visual box size=0.47245005204754464 0.3340878974221754 0.11994987425580875
- link Link5: geometry collision box size=0.8531426075040301 0.9979130014617206 0.10848934102777089; visual box size=0.8531426075040301 0.9979130014617206 0.10848934102777089
- link Link6: geometry collision box size=0.19222018618823225 0.9277426351632009 1.024797929856107; visual box size=0.19222018618823225 0.9277426351632009 1.024797929856107
Joints:
- removed joint Link10_Link11
- removed joint Link11_Link12
- removed joint Link6_Link7
- removed joint Link7_Link8
- removed joint Link8_Link9
- removed joint Link9_Link10
- joint Link0_Link1: origin xyz=-1 -0.35754571454787576 0.5 rpy=0 0 0 -> xyz=-0.8768316047916612 0 0.5 rpy=0 0 0
- joint Link1_Link2: origin xyz=0 0.6976178794959438 0 rpy=0 0 0 -> xyz=0.37097230349296273 -0.27316728774679455 0 rpy=0 0 0
- joint Link2_Link3: origin xyz=0 0.8369508294019093 0 rpy=0 0 0 -> xyz=-0.18770213318240098 -0.3927514969129071 0 rpy=0 0 0
- joint Link3_Link4: origin xyz=0.2670114302747143 0.24985912281608025 0 rpy=0 0 0 -> xyz=-0.31098733205897927 0.10916798355357384 0 rpy=0 0 0
- joint Link4_Link5: origin xyz=0.5290775594231117 0.24771301442539811 0 rpy=0 0 0 -> xyz=0 0.3340878974221754 0 rpy=0 0 0
- joint Link5_Link6: origin xyz=0 0.8848313811778493 0 rpy=0 0 0 -> xyz=-0.4265713037520151 0.4989565007308603 0 rpy=0 0 0

Commit message: fitness errors

File: body.urdf (robot description, URDF)
Before this commit: robot robot, 7 links, 6 joints
Links:
- removed link Link5
- removed link Link6
- link Link0: geometry collision box size=0.11718924006925083 0.7301109981024647 0.11212437219628438; visual box size=0.11718924006925083 0.7301109981024647 0.11212437219628438
- link Link1: geometry collision box size=0.2561606918905849 0.6640921782415155 0.6097142751099945; visual box size=0.2561606918905849 0.6640921782415155 0.6097142751099945
- link Link2: geometry collision box size=0.8211544167805355 0.12352374299330429 0.4517559389217146; visual box size=0.8211544167805355 0.12352374299330429 0.4517559389217146
- link Link3: geometry collision box size=0.8496428283489856 0.23796208142151723 0.46847675033122804; visual box size=0.8496428283489856 0.23796208142151723 0.46847675033122804
- link Link4: geometry collision box size=0.6841838813547958 0.17127896451442307 0.7630423142707581; visual box size=0.6841838813547958 0.17127896451442307 0.7630423142707581
Joints:
- removed joint Link4_Link5
- removed joint Link5_Link6
- joint Link0_Link1: origin xyz=-0.8768316047916612 0 0.5 rpy=0 0 0 -> xyz=-1.0585946200346255 0 0.5 rpy=0 0 0
- joint Link1_Link2: origin xyz=0.37097230349296273 -0.27316728774679455 0 rpy=0 0 0 -> xyz=-0.12808034594529244 0.3320460891207577 0 rpy=0 0 0
- joint Link2_Link3: origin xyz=-0.18770213318240098 -0.3927514969129071 0 rpy=0 0 0 -> xyz=0 0.12352374299330429 0 rpy=0 0 0
- joint Link3_Link4: origin xyz=-0.31098733205897927 0.10916798355357384 0 rpy=0 0 0 -> xyz=-0.4248214141744928 0.11898104071075861 0 rpy=0 0 0
