Commit message: need to manually run seeds

File: body0.urdf (robot description, URDF)
Before this commit: robot robot, 5 links, 4 joints
Links:
- removed link Link4
- link Link0: geometry collision box size=0.4689255239026796 0.16190914471997989 1.002927011249925; visual box size=0.4689255239026796 0.16190914471997989 1.002927011249925
- link Link1: geometry collision box size=1.0035276283933792 0.733140454933967 0.21067593107723906; visual box size=1.0035276283933792 0.733140454933967 0.21067593107723906
- link Link2: geometry collision box size=0.9442205703700911 0.12910574128749155 0.9725666902442477; visual box size=0.9442205703700911 0.12910574128749155 0.9725666902442477
- link Link3: geometry collision box size=0.6031018261359922 0.5040569596579633 1.0464135665518512; visual box size=0.6031018261359922 0.5040569596579633 1.0464135665518512
Joints:
- removed joint Link3_Link4
- joint Link0_Link1: origin xyz=-1 0.4947023969044642 0.5 rpy=0 0 0 -> xyz=-1 -0.08095457235998994 0.5 rpy=0 0 0
- joint Link1_Link2: origin xyz=0 -1.0693618542741905 0 rpy=0 0 0 -> xyz=0.5017638141966896 0.3665702274669835 0 rpy=0 0 0
- joint Link2_Link3: origin xyz=0.5193199744390917 -0.4115368700167693 0 rpy=0 0 0 -> xyz=0.9442205703700911 0 0 rpy=0 0 0

Commit message: not working!

File: body0.urdf (robot description, URDF)
Before this commit: robot robot, 4 links, 3 joints
Links:
- removed link Link3
- link Link0: geometry collision box size=1.016313958871695 0.38814045461294244 0.4285205894100186; visual box size=1.016313958871695 0.38814045461294244 0.4285205894100186
- link Link1: geometry collision box size=0.3360608100428363 0.36313055635157665 0.9991573739349746; visual box size=0.3360608100428363 0.36313055635157665 0.9991573739349746
- link Link2: geometry collision box size=0.3749746019982261 0.16152146230112222 0.6451022718292647; visual box size=0.3749746019982261 0.16152146230112222 0.6451022718292647
Joints:
- removed joint Link2_Link3
- joint Link0_Link1: origin xyz=-1 -0.08095457235998994 0.5 rpy=0 0 0 -> xyz=-1 0 0.7142602947050093 rpy=0 0 0
- joint Link1_Link2: origin xyz=0.5017638141966896 0.3665702274669835 0 rpy=0 0 0 -> xyz=0 0 0.9991573739349746 rpy=0 0 0

Commit message: making changes

File: body0.urdf (robot description, URDF)
Before this commit: robot robot, 3 links, 2 joints
Links:
- added link Link3, mass 1; collision box size=1.0840756553192437 0.6566033596330159 0.5520899308663075; visual box size=1.0840756553192437 0.6566033596330159 0.5520899308663075
- added link Link4, mass 1; collision box size=0.14519020587278178 0.27204972098548574 1.0484359838390518; visual box size=0.14519020587278178 0.27204972098548574 1.0484359838390518
- added link Link5, mass 1; collision box size=1.0957803178738903 0.5733710133409355 0.7253416791036114; visual box size=1.0957803178738903 0.5733710133409355 0.7253416791036114
- added link Link6, mass 1; collision box size=0.8072784462317724 0.42006242494792456 0.9699951765427978; visual box size=0.8072784462317724 0.42006242494792456 0.9699951765427978
- link Link0: geometry collision box size=0.9404529137648749 0.23019248875762469 1.0859838701204876; visual box size=0.9404529137648749 0.23019248875762469 1.0859838701204876
- link Link1: geometry collision box size=0.6551190239538548 0.9620262961060153 0.6461180824058927; visual box size=0.6551190239538548 0.9620262961060153 0.6461180824058927
- link Link2: geometry collision box size=1.0302360252589933 0.17283153459015968 0.4171161096588637; visual box size=1.0302360252589933 0.17283153459015968 0.4171161096588637
Joints:
- added joint Link2_Link3: type revolute, parent Link2, child Link3, origin xyz=0.5151180126294966 0 0.20855805482943185 rpy=0 0 0, axis 1 0 0, limit lower=-3.14159 upper=3.14159 effort=0.0 velocity=0.0
- added joint Link3_Link4: type revolute, parent Link3, child Link4, origin xyz=0.5420378276596218 0 0.27604496543315377 rpy=0 0 0, axis 1 0 0, limit lower=-3.14159 upper=3.14159 effort=0.0 velocity=0.0
- added joint Link4_Link5: type revolute, parent Link4, child Link5, origin xyz=0.07259510293639089 -0.13602486049274287 0 rpy=0 0 0, axis 1 0 0, limit lower=-3.14159 upper=3.14159 effort=0.0 velocity=0.0
- added joint Link5_Link6: type revolute, parent Link5, child Link6, origin xyz=0 -0.28668550667046777 0.3626708395518057 rpy=0 0 0, axis 1 0 0, limit lower=-3.14159 upper=3.14159 effort=0.0 velocity=0.0
- joint Link0_Link1: origin xyz=-1 0 0.7142602947050093 rpy=0 0 0 -> xyz=-1 0.11509624437881234 0.5 rpy=0 0 0
- joint Link1_Link2: origin xyz=0 0 0.9991573739349746 rpy=0 0 0 -> xyz=0.3275595119769274 -0.48101314805300766 0 rpy=0 0 0

Commit message: issues

File: body0.urdf (robot description, URDF)
Before this commit: robot robot, 7 links, 6 joints
Links:
- removed link Link5
- removed link Link6
- link Link0: geometry collision box size=0.2495688533681291 0.6317293571780894 0.9039777950740041; visual box size=0.2495688533681291 0.6317293571780894 0.9039777950740041
- link Link1: geometry collision box size=0.6143703257861456 0.20307286089689838 0.70296337089398; visual box size=0.6143703257861456 0.20307286089689838 0.70296337089398
- link Link2: geometry collision box size=0.6747188857218435 0.6580261867397467 0.658801451178701; visual box size=0.6747188857218435 0.6580261867397467 0.658801451178701
- link Link3: geometry collision box size=0.5347536331170385 1.030213366481426 1.0553170734559885; visual box size=0.5347536331170385 1.030213366481426 1.0553170734559885
- link Link4: geometry collision box size=0.5945753896680066 0.433242556344403 0.6437988073382573; visual box size=0.5945753896680066 0.433242556344403 0.6437988073382573
Joints:
- removed joint Link4_Link5
- removed joint Link5_Link6
- joint Link0_Link1: origin xyz=-1 0.11509624437881234 0.5 rpy=0 0 0 -> xyz=-1 0 0.9519888975370021 rpy=0 0 0
- joint Link1_Link2: origin xyz=0.3275595119769274 -0.48101314805300766 0 rpy=0 0 0 -> xyz=0 0.10153643044844919 0.35148168544699 rpy=0 0 0
- joint Link2_Link3: origin xyz=0.5151180126294966 0 0.20855805482943185 rpy=0 0 0 -> xyz=0 0.32901309336987333 0.3294007255893505 rpy=0 0 0
- joint Link3_Link4: origin xyz=0.5420378276596218 0 0.27604496543315377 rpy=0 0 0 -> xyz=-0.26737681655851925 0 0.5276585367279942 rpy=0 0 0

Commit message: making progress

File: body0.urdf (robot description, URDF)
Before this commit: robot robot, 5 links, 4 joints
Links:
- removed link Link3
- removed link Link4
- link Link0: geometry collision box size=0.4806444878411589 0.8292154535957873 0.6978739053635076; visual box size=0.4806444878411589 0.8292154535957873 0.6978739053635076
- link Link1: geometry collision box size=0.7567753156562895 0.9293005158642262 0.5107851315249385; visual box size=0.7567753156562895 0.9293005158642262 0.5107851315249385
- link Link2: geometry collision box size=0.1350879387840679 0.8489349187102823 0.9514488458044126; visual box size=0.1350879387840679 0.8489349187102823 0.9514488458044126
Joints:
- removed joint Link2_Link3
- removed joint Link3_Link4
- joint Link0_Link1: origin xyz=-1 0 0.9519888975370021 rpy=0 0 0 -> xyz=-1.2403222439205794 0 0.5 rpy=0 0 0
- joint Link1_Link2: origin xyz=0 0.10153643044844919 0.35148168544699 rpy=0 0 0 -> xyz=-0.37838765782814476 0.4646502579321131 0 rpy=0 0 0

Commit message: finishing a8

File: body0.urdf (robot description, URDF)
Before this commit: robot robot, 3 links, 2 joints
Links:
- link Link0: geometry collision box size=0.7583072849102449 0.40421192212862533 0.45055647096616636; visual box size=0.7583072849102449 0.40421192212862533 0.45055647096616636
- link Link1: geometry collision box size=0.8135990507986669 0.7480779070521546 0.2342665386094879; visual box size=0.8135990507986669 0.7480779070521546 0.2342665386094879
- link Link2: geometry collision box size=0.4982858371808703 0.8757839427301374 0.10817493532044634; visual box size=0.4982858371808703 0.8757839427301374 0.10817493532044634
Joints:
- joint Link0_Link1: origin xyz=-1.2403222439205794 0 0.5 rpy=0 0 0 -> xyz=-0.6208463575448775 0 0.5 rpy=0 0 0
- joint Link1_Link2: origin xyz=-0.37838765782814476 0.4646502579321131 0 rpy=0 0 0 -> xyz=0.8135990507986669 0 0 rpy=0 0 0

File: body1.urdf (robot description, URDF)
Before this commit: robot robot, 3 links, 2 joints
Links:
- added link Link3, mass 1; collision box size=0.7389691811162546 0.8441562806815373 0.8166649400429331; visual box size=0.7389691811162546 0.8441562806815373 0.8166649400429331
- link Link0: geometry collision box size=0.7583072849102449 0.40421192212862533 0.45055647096616636; visual box size=0.7583072849102449 0.40421192212862533 0.45055647096616636
- link Link1: geometry collision box size=0.8135990507986669 0.7480779070521546 0.2342665386094879; visual box size=0.8135990507986669 0.7480779070521546 0.2342665386094879
- link Link2: geometry collision box size=0.4982858371808703 0.8757839427301374 0.10817493532044634; visual box size=0.4982858371808703 0.8757839427301374 0.10817493532044634
Joints:
- added joint Link2_Link3: type revolute, parent Link2, child Link3, origin xyz=0.24914291859043514 0.4378919713650687 0 rpy=0 0 0, axis 1 0 0, limit lower=-3.14159 upper=3.14159 effort=0.0 velocity=0.0
- joint Link0_Link1: origin xyz=-1 0.31307029436997363 0.5 rpy=0 0 0 -> xyz=-0.6208463575448775 0 0.5 rpy=0 0 0
- joint Link1_Link2: origin xyz=0 -0.9895005000467663 0 rpy=0 0 0 -> xyz=0.8135990507986669 0 0 rpy=0 0 0
