Commit message: final submission

File: body11.urdf (robot description, URDF)
Before this commit: robot robot, 3 links, 2 joints
Links:
- added link Link3, mass 1; collision box size=0.16551442597523927 0.3796358445809499 0.8353614517017636; visual box size=0.16551442597523927 0.3796358445809499 0.8353614517017636
Joints:
- added joint Link2_Link3: type revolute, parent Link2, child Link3, origin xyz=0.343818130999691 0 0.4050162302520329 rpy=0 0 0, axis 1 0 0, limit lower=-3.14159 upper=3.14159 effort=0.0 velocity=0.0

File: body14.urdf (robot description, URDF)
Before this commit: robot robot, 3 links, 2 joints
Links:
- link Link0: geometry collision box size=0.782837624497281 0.6433287656324278 0.4202571989295951; visual box size=0.782837624497281 0.6433287656324278 0.4202571989295951
- link Link1: geometry collision box size=0.22668774356900726 1.0673855422523317 0.9751826674099321; visual box size=0.22668774356900726 1.0673855422523317 0.9751826674099321
- link Link2: geometry collision box size=0.6169934303937662 0.5968063664221731 0.330077150702593; visual box size=0.6169934303937662 0.5968063664221731 0.330077150702593
Joints:
- joint Link0_Link1: origin xyz=-1 -0.33603531213612664 0.5 rpy=0 0 0 -> xyz=-0.6085811877513595 0 0.5 rpy=0 0 0
- joint Link1_Link2: origin xyz=0.3686353301408588 0.360850606672044 0 rpy=0 0 0 -> xyz=0.22668774356900726 0 0 rpy=0 0 0

File: body19.urdf (robot description, URDF)
Before this commit: robot robot, 3 links, 2 joints
Links:
- link Link0: geometry collision box size=0.6652890909741219 0.8009669814799684 0.7199866284384536; visual box size=0.6652890909741219 0.8009669814799684 0.7199866284384536
- link Link1: geometry collision box size=0.5900380781581765 1.0486795332152736 0.46930296620953826; visual box size=0.5900380781581765 1.0486795332152736 0.46930296620953826
- link Link2: geometry collision box size=0.4943180123338511 0.3887392213116384 0.7801257478087449; visual box size=0.4943180123338511 0.3887392213116384 0.7801257478087449
Joints:
- joint Link0_Link1: origin xyz=-1 -0.33603531213612664 0.5 rpy=0 0 0 -> xyz=-1.332644545487061 0 0.5 rpy=0 0 0
- joint Link1_Link2: origin xyz=0.3686353301408588 0.360850606672044 0 rpy=0 0 0 -> xyz=-0.2950190390790883 0.5243397666076368 0 rpy=0 0 0

File: body2.urdf (robot description, URDF)
Before this commit: robot robot, 3 links, 2 joints
Links:
- link Link0: geometry collision box size=0.5367457924623316 0.3662525450869899 0.9101788082727653; visual box size=0.5367457924623316 0.3662525450869899 0.9101788082727653
- link Link1: geometry collision box size=0.7700421531535787 0.39280551092624627 0.7760914331195407; visual box size=0.7700421531535787 0.39280551092624627 0.7760914331195407
- link Link2: geometry collision box size=0.7262537740893681 0.11726963809980365 0.6167988491530254; visual box size=0.7262537740893681 0.11726963809980365 0.6167988491530254
Joints:
- joint Link0_Link1: origin xyz=-1 -0.33603531213612664 0.5 rpy=0 0 0 -> xyz=-1 -0.18312627254349495 0.5 rpy=0 0 0
- joint Link1_Link2: origin xyz=0.3686353301408588 0.360850606672044 0 rpy=0 0 0 -> xyz=0 0.39280551092624627 0 rpy=0 0 0

File: body3.urdf (robot description, URDF)
Before this commit: robot robot, 3 links, 2 joints
Links:
- link Link0: geometry collision box size=0.35771127395562585 0.33768191152544436 0.23693453941081724; visual box size=0.35771127395562585 0.33768191152544436 0.23693453941081724
- link Link1: geometry collision box size=0.21098904258987441 0.9021420738250111 0.4701826042577838; visual box size=0.21098904258987441 0.9021420738250111 0.4701826042577838
- link Link2: geometry collision box size=1.0807504560984382 0.13326428278307537 0.3336879244632639; visual box size=1.0807504560984382 0.13326428278307537 0.3336879244632639
Joints:
- joint Link0_Link1: origin xyz=-1 -0.33603531213612664 0.5 rpy=0 0 0 -> xyz=-1 0 0.6184672697054087 rpy=0 0 0
- joint Link1_Link2: origin xyz=0.3686353301408588 0.360850606672044 0 rpy=0 0 0 -> xyz=0.10549452129493721 0 0.2350913021288919 rpy=0 0 0

File: body5.urdf (robot description, URDF)
Before this commit: robot robot, 3 links, 2 joints
Links:
- link Link0: geometry collision box size=0.8070058863139927 0.8860161182149293 0.18690123502180714; visual box size=0.8070058863139927 0.8860161182149293 0.18690123502180714
- link Link1: geometry collision box size=0.6875169993630148 0.13692808679283933 0.9487766677980467; visual box size=0.6875169993630148 0.13692808679283933 0.9487766677980467
- link Link2: geometry collision box size=0.4331568240854953 0.14693459938798217 1.0874925323303313; visual box size=0.4331568240854953 0.14693459938798217 1.0874925323303313
Joints:
- joint Link0_Link1: origin xyz=-1 -0.33603531213612664 0.5 rpy=0 0 0 -> xyz=-1 -0.44300805910746466 0.5 rpy=0 0 0
- joint Link1_Link2: origin xyz=0.3686353301408588 0.360850606672044 0 rpy=0 0 0 -> xyz=0.3437584996815074 0.06846404339641966 0 rpy=0 0 0

File: body6.urdf (robot description, URDF)
Before this commit: robot robot, 3 links, 2 joints
Links:
- link Link0: geometry collision box size=0.8768034244302926 0.44547554503646736 0.12078494021382905; visual box size=0.8768034244302926 0.44547554503646736 0.12078494021382905
- link Link1: geometry collision box size=0.9721575899729865 0.34157470764235687 0.9719372961252903; visual box size=0.9721575899729865 0.34157470764235687 0.9719372961252903
- link Link2: geometry collision box size=0.20126792387427897 0.6746613637427691 0.11745544231318963; visual box size=0.20126792387427897 0.6746613637427691 0.11745544231318963
Joints:
- joint Link0_Link1: origin xyz=-1 -0.33603531213612664 0.5 rpy=0 0 0 -> xyz=-1 0.22273777251823368 0.5 rpy=0 0 0
- joint Link1_Link2: origin xyz=0.3686353301408588 0.360850606672044 0 rpy=0 0 0 -> xyz=0 -0.34157470764235687 0 rpy=0 0 0

File: body7.urdf (robot description, URDF)
Before this commit: robot robot, 3 links, 2 joints
Links:
- link Link0: geometry collision box size=0.9443342778423313 0.926257625132848 0.34799147213706816; visual box size=0.9443342778423313 0.926257625132848 0.34799147213706816
- link Link1: geometry collision box size=0.16504441698579278 0.12076766765515792 0.3687765950421993; visual box size=0.16504441698579278 0.12076766765515792 0.3687765950421993
- link Link2: geometry collision box size=0.5207472410395759 1.0079768298804563 0.2608278168029242; visual box size=0.5207472410395759 1.0079768298804563 0.2608278168029242
Joints:
- joint Link0_Link1: origin xyz=-1 -0.33603531213612664 0.5 rpy=0 0 0 -> xyz=-1.4721671389211657 0 0.5 rpy=0 0 0
- joint Link1_Link2: origin xyz=0.3686353301408588 0.360850606672044 0 rpy=0 0 0 -> xyz=-0.08252220849289639 -0.06038383382757896 0 rpy=0 0 0

File: body8.urdf (robot description, URDF)
Before this commit: robot robot, 3 links, 2 joints
Links:
- link Link0: geometry collision box size=0.34764086893317525 0.7112101920520445 0.9460897671316999; visual box size=0.34764086893317525 0.7112101920520445 0.9460897671316999
- link Link1: geometry collision box size=0.28251203114446477 0.8662040772961432 0.543737230293859; visual box size=0.28251203114446477 0.8662040772961432 0.543737230293859
- link Link2: geometry collision box size=0.24349033653645372 0.3924458990801378 0.19991876880380213; visual box size=0.24349033653645372 0.3924458990801378 0.19991876880380213
Joints:
- joint Link0_Link1: origin xyz=-1 -0.33603531213612664 0.5 rpy=0 0 0 -> xyz=-1.1738204344665877 0 0.5 rpy=0 0 0
- joint Link1_Link2: origin xyz=0.3686353301408588 0.360850606672044 0 rpy=0 0 0 -> xyz=-0.14125601557223239 0 0.2718686151469295 rpy=0 0 0
